Commit message: Adding battery, camera and hokuyo to the model TODO: topic're not working

File: meine_bot/urdf/meine_bot.xacro (robot description, xacro)
@@ -36,9 +36,88 @@
       </geometry>
     </visual>
+    <xacro:default_inertial mass="5"/>
+  </link>
+  <link name="battery">
+    <visual>
+      <origin xyz="0 0 0" rpy="0 0 ${pi/2}"/>
+      <geometry>
+        <box size="${battery_length} ${battery_width} ${battery_height}"/>
+      </geometry>
+    </visual>
+    <collision>
+      <origin xyz="0 0 0" rpy="0 0 ${pi/2}"/>
+      <geometry>
+        <box size="${battery_length} ${battery_width} ${battery_height}"/>
+      </geometry>
+    </collision>
     <xacro:default_inertial mass="10"/>
   </link>
+  <joint name="battery_chassi_joint" type="fixed">
+    <origin xyz="${length/2 - battery_width/2} 0 ${battery_height/2}" rpy="0 0 0" />
+    <parent link="chassis"/>
+      <child link="battery"/>
+  </joint>
   <xacro:motor_default name="left" reflect="1"/>
   <xacro:motor_default name="right" reflect="-1"/>
   <xacro:wheel_default name="left" reflect="1"/>
   <xacro:wheel_default name="right" reflect="-1"/>
+  <link name="camera">
+    <inertial>
+      <mass value ="0.1"/>
+      <origin xyz="0 0 0" rpy="0 0 0"/>
+      <inertia
+        ixx="1e-6" ixy="0" ixz="0"
+        iyy="1e-6" iyz="0"
+        izz="1e-6"
+      />
+    </inertial>
+    <collision name="collision">
+      <origin xyz="0 0 0" rpy="0 0 0"/>
+      <geometry>
+        <box size="${camera_length} ${camera_width} ${camera_height}"/>
+      </geometry>
+    </collision>
+    <visual name='camera_visual'>
+      <origin xyz="0 0 0" rpy="0 0 0"/>
+      <geometry>
+        <box size="${camera_length} ${camera_width} ${camera_height}"/>
+      </geometry>
+      <material name="">
+          <color rgba="0 0 1 0.5"/>
+      </material>
+    </visual>
+  </link>
+  <joint name="camera_joint" type="fixed">
+    <origin xyz="${-length/2} 0 ${-camera_height /2}" rpy="0 0 0"/>
+    <parent link="chassis"/>
+    <child link="camera" />
+  </joint>
+  <link name="hokuyo">
+    <inertial>
+      <mass value ="0.1"/>
+      <origin xyz="0 0 0" rpy="0 0 0"/>
+      <inertia
+        ixx="1e-6" ixy="0" ixz="0"
+        iyy="1e-6" iyz="0"
+        izz="1e-6"
+      />
+    </inertial>
+    <collision name="collision">
+      <origin xyz="0 0 0" rpy="0 0 0"/>
+      <geometry>
+        <box size="${hokuyo_width} ${hokuyo_width} ${hokuyo_width}"/>
+      </geometry>
+    </collision>
+    <visual name='hokuyo_visual'>
+      <origin xyz="0 0 0" rpy="0 0 0"/>
+      <geometry>
+        <mesh filename="package://udacity_bot/meshes/hokuyo.dae"/>
+      </geometry>
+    </visual>
+  </link>
+  <joint name="hokuyo_joint" type="fixed">
+    <origin xyz="${-length/2 + hokuyo_width / 2} 0 ${hokuyo_width/2}" rpy="0 0 0"/>
+    <parent link="chassis"/>
+    <child link="hokuyo" />
+  </joint>
 </robot>

File: meine_bot/urdf/meine_bot_values.xacro (robot description, xacro)
@@ -13,4 +13,14 @@
   <xacro:property name="y_pos" value="${width/2 - motor_width/2}"/>
   <xacro:property name="z_pos" value="${-motor_height/2}"/>
+  <!-- BATTERY AND PI -->
+  <xacro:property name="battery_width" value="0.065"/>
+  <xacro:property name="battery_length" value="0.11"/>
+  <xacro:property name="battery_height" value="0.05"/>
+  <!-- CAMERA -->
+  <xacro:property name="camera_width" value="0.03"/>
+  <xacro:property name="camera_length" value="0.03"/>
+  <xacro:property name="camera_height" value="0.02"/>
+  <!-- CAMERA -->
+  <xacro:property name="hokuyo_width" value="0.1"/>
   <!-- CASTER-->
   <xacro:property name="radius_caster" value="0.01725"/>

Commit message: swap robot direction

File: meine_bot/urdf/meine_bot.xacro (robot description, xacro)
@@ -5,4 +5,5 @@
   <!-- IF YOU WANT CHANGE SOME BEHAVIOR FROM THE INERTIAL OR WHEEL SEE THIS FILE-->
   <xacro:include filename="$(find meine_bot)/urdf/meine_bot_macros.xacro"/>
+  <xacro:include filename="$(find meine_bot)/urdf/meine_bot.gazebo"/>
   <link name="robot_footprint"></link>
   <joint name="robot_footprint_joint" type="fixed">
@@ -25,5 +26,5 @@
     </collision>
     <collision name='back_caster_collision'>
-      <origin xyz="${length/2} 0 ${-radius_caster} " rpy=" 0 0 0"/>
+      <origin xyz="${-length/2} 0 ${-radius_caster} " rpy=" 0 0 0"/>
       <geometry>
         <sphere radius="${radius_caster - 0.0001}"/>
@@ -31,5 +32,5 @@
     </collision>
     <visual name='back_caster_visual'>
-      <origin xyz="${length/2} 0 ${-radius_caster} " rpy=" 0 0 0"/>
+      <origin xyz="${-length/2} 0 ${-radius_caster} " rpy=" 0 0 0"/>
       <geometry>
         <sphere radius="${radius_caster}"/>
@@ -54,5 +55,5 @@
   </link>
   <joint name="battery_chassi_joint" type="fixed">
-    <origin xyz="${length/2 - battery_width/2} 0 ${battery_height/2}" rpy="0 0 0" />
+    <origin xyz="${- length/2 + battery_width/2} 0 ${battery_height/2}" rpy="0 0 0" />
     <parent link="chassis"/>
       <child link="battery"/>
@@ -89,5 +90,5 @@
   </link>
   <joint name="camera_joint" type="fixed">
-    <origin xyz="${-length/2} 0 ${-camera_height /2}" rpy="0 0 0"/>
+    <origin xyz="${length/2} 0 ${-camera_height /2}" rpy="0 0 0"/>
     <parent link="chassis"/>
     <child link="camera" />
@@ -117,5 +118,5 @@
   </link>
   <joint name="hokuyo_joint" type="fixed">
-    <origin xyz="${-length/2 + hokuyo_width / 2} 0 ${hokuyo_width/2}" rpy="0 0 0"/>
+    <origin xyz="${length/2 - hokuyo_width / 2} 0 ${hokuyo_width/2}" rpy="0 0 0"/>
     <parent link="chassis"/>
     <child link="hokuyo" />

File: meine_bot/urdf/meine_bot_macros.xacro (robot description, xacro)
@@ -59,5 +59,5 @@
     </link>
     <joint name="motor_${name}_hinge" type="fixed">
-      <origin xyz="${x_pos} ${reflect * y_pos} ${z_pos}" rpy="0 0 0" />
+      <origin xyz="${-x_pos} ${reflect * y_pos} ${z_pos}" rpy="0 0 0" />
       <parent link="chassis"/>
       <child link='motor_${name}'  />

Commit message: changing the hokuyo position and adding some colors

File: meine_bot/urdf/meine_bot.xacro (robot description, xacro)
@@ -52,5 +52,5 @@
       </geometry>
     </collision>
-    <xacro:default_inertial mass="10"/>
+    <xacro:default_inertial mass="5"/>
   </link>
   <joint name="battery_chassi_joint" type="fixed">
@@ -118,5 +118,5 @@
   </link>
   <joint name="hokuyo_joint" type="fixed">
-    <origin xyz="${length/2 - hokuyo_width / 2} 0 ${hokuyo_width/2}" rpy="0 0 0"/>
+    <origin xyz="${length/2 } 0 ${hokuyo_width/2}" rpy="0 0 0"/>
     <parent link="chassis"/>
     <child link="hokuyo" />

File: meine_bot/urdf/meine_bot_macros.xacro (robot description, xacro)
@@ -54,5 +54,5 @@
         </geometry>
         <material name="yellow">
-          <color rgba="0 1 1 1"/>
+          <color rgba="1 1 0 1"/>
         </material>
       </visual>

Commit message: Adding Mass variables

File: meine_bot/urdf/meine_bot.xacro (robot description, xacro)
@@ -37,5 +37,5 @@
       </geometry>
     </visual>
-    <xacro:default_inertial mass="5"/>
+    <xacro:default_inertial mass="${chassi_mass}"/>
   </link>
   <link name="battery">
@@ -52,5 +52,5 @@
       </geometry>
     </collision>
-    <xacro:default_inertial mass="5"/>
+    <xacro:default_inertial mass="${battery_mass}"/>
   </link>
   <joint name="battery_chassi_joint" type="fixed">

File: meine_bot/urdf/meine_bot_macros.xacro (robot description, xacro)
@@ -14,5 +14,5 @@
   <xacro:macro name="wheel_default" params="name reflect">
     <link name='wheel_${name}'>
-      <xacro:default_inertial mass="5"/>
+      <xacro:default_inertial mass="${wheel_mass}"/>
       <collision name='wheel_${name}_collision'>
         <origin xyz="0 ${reflect * motor_width} 0" rpy="0 ${reflect * pi/2} ${reflect * pi/2} "/>

File: meine_bot/urdf/meine_bot_values.xacro (robot description, xacro)
@@ -6,4 +6,5 @@
   <xacro:property name="length" value="0.2"/>
   <xacro:property name="height" value="0.0002"/>
+  <xacro:property name="chassi_mass" value="5"/>
   <!-- MOTOR -->
   <xacro:property name="motor_width" value="0.02"/>
@@ -17,9 +18,10 @@
   <xacro:property name="battery_length" value="0.11"/>
   <xacro:property name="battery_height" value="0.05"/>
+  <xacro:property name="battery_mass" value="5"/>
   <!-- CAMERA -->
   <xacro:property name="camera_width" value="0.03"/>
   <xacro:property name="camera_length" value="0.03"/>
   <xacro:property name="camera_height" value="0.02"/>
-  <!-- CAMERA -->
+  <!-- HOKUYO -->
   <xacro:property name="hokuyo_width" value="0.1"/>
   <!-- CASTER-->
@@ -28,4 +30,5 @@
   <xacro:property name="radius_wheel" value="0.03"/>
   <xacro:property name="length_wheel" value="0.025"/>
+  <xacro:property name="wheel_mass" value="5"/>
   <!-- INERTIA-->
   <xacro:property name='inertial' value="0.1"/>
