Commit message: Adding some space between chassi and wheels

File: meine_bot/urdf/meine_bot_macros.xacro (robot description, xacro)
@@ -32,5 +32,5 @@
     </link>
     <joint name="wheel_${name}_hinge" type="continuous">
-      <origin xyz="0 0 ${z_pos}" rpy="0 0 0" />
+      <origin xyz="0 ${reflect * 0.01} ${z_pos}" rpy="0 0 0" />
       <parent link="motor_${name}"/>
       <child link='wheel_${name}'  />

Commit message: changing the frinction and damping

File: meine_bot/urdf/meine_bot_macros.xacro (robot description, xacro)
@@ -36,5 +36,5 @@
       <child link='wheel_${name}'  />
       <axis xyz="0 1 0" rpy="0 0 0"/>
-      <dynamics damping="1.0" friction="1.0"/>
+      <dynamics damping=".01" friction=".01"/>
     </joint>
   </xacro:macro>
